Commit message: Leg

File: description/robot_core.xacro (robot description, xacro)
@@ -17,87 +17,65 @@
     <link name="base_link">
     </link>
-    <!-- CHASSIS LINK -->
-    <joint name="chassis_joint" type="fixed">
+    <!-- FOOT LINK -->
+    <joint name="foot_joint" type="fixed">
         <parent link="base_link"/>
-        <child link="chassis"/>
-        <origin xyz="-0.1 0 0"/>
-    </joint>
-    <link name="chassis">
-        <visual>
-            <origin xyz="0.15 0 0.075"/>
-            <geometry>
-                <box size="0.3 0.3 0.15"/>
-            </geometry>
-            <material name="white"/>
-        </visual>
-        <collision>
-            <origin xyz="0.15 0 0.075"/>
-            <geometry>
-                <box size="0.3 0.3 0.15"/>
-            </geometry>
-            <material name="white"/>
-        </collision>
-        <xacro:inertial_box mass="0.5" x="0.3" y="0.3" z="0.15">
-            <origin xyz="0.15 0 0.075" rpy="0 0 0"/>
-        </xacro:inertial_box>
-    </link>
-    <!-- LEFT WHEEL LINK -->
-    <joint name="left_wheel_joint" type="continuous">
-        <parent link="base_link"/>
-        <child link="left_wheel"/>
-        <origin xyz="0 0.175 0" rpy="-${pi/2} 0 0"/>
-        <axis xyz="0 0 1"/>
-    </joint>
-    <link name="left_wheel">
-        <visual>
-            <geometry>
-                <cylinder radius="0.05" length="0.04"/>
-            </geometry>
-            <material name="blue"/>
-        </visual>
-        <collision>
-            <geometry>
-                <cylinder radius="0.05" length="0.04"/>
-            </geometry>
-            <material name="blue"/>
-        </collision>
-        <xacro:inertial_cylinder mass="0.1" radius="0.05" length="0.04">
-            <origin xyz="0 0 0" rpy="0 0 0"/>
-        </xacro:inertial_cylinder>
-    </link>
-    <!-- RIGHT WHEEL LINK -->
-    <joint name="right_wheel_joint" type="continuous">
-        <parent link="base_link"/>
-        <child link="right_wheel"/>
-        <origin xyz="0 -0.175 0" rpy="${pi/2} 0 0"/>
-        <axis xyz="0 0 -1"/>
-    </joint>
-    <link name="right_wheel">
-        <visual>
-            <geometry>
-                <cylinder radius="0.05" length="0.04"/>
-            </geometry>
-            <material name="blue"/>
-        </visual>
-        <collision>
-            <geometry>
-                <cylinder radius="0.05" length="0.04"/>
-            </geometry>
-            <material name="blue"/>
-        </collision>
-        <xacro:inertial_cylinder mass="0.1" radius="0.05" length="0.04">
-            <origin xyz="0 0 0" rpy="0 0 0"/>
-        </xacro:inertial_cylinder>
-    </link>
-    <!-- CASTER WHEEL LINK -->
-    <joint name="caster_wheel_joint" type="fixed">
-        <parent link="chassis"/>
-        <child link="caster_wheel"/>
-        <origin xyz="0.24 0 0"/>
-    </joint>
-    <link name="caster_wheel">
-        <visual>
-            <geometry>
-                <sphere radius="0.05"/>
+        <child link="foot"/>
+        <origin xyz="-0.05 0 0"/>
+        <axis xyz="0 1 1"/>
+    </joint>
+    <link name="foot">
+        <visual>
+            <origin xyz="0.05 0 0.01"/>
+            <geometry>
+                <box size="0.1 0.05 0.02"/>
+            </geometry>
+            <material name="white"/>
+        </visual>
+        <collision>
+            <origin xyz="0.05 0 0.01"/>
+            <geometry>
+                <box size="0.1 0.05 0.02"/>
+            </geometry>
+            <material name="white"/>
+        </collision>
+        <!-- <xacro:inertial_box mass="0.5" x="0.3" y="0.3" z="0.15"> -->
+            <!-- <origin xyz="0.15 0 0.075" rpy="0 0 0"/> -->
+        <!-- </xacro:inertial_box> -->
+    </link>
+    <!-- ANKLE_YAW LINK -->
+    <joint name="ankle_yaw_joint" type="continuous">
+        <parent link="foot"/>
+        <child link="ankle_yaw"/>
+        <origin xyz="-0.01 0 0.01" rpy="0 0 0"/>
+        <axis xyz="0 0 1"/>
+    </joint>
+    <link name="ankle_yaw">
+        <visual>
+            <geometry>
+                <cylinder radius="0.01" length="0.01"/>
+            </geometry>
+            <material name="blue"/>
+        </visual>
+        <collision>
+            <geometry>
+                <cylinder radius="0.01" length="0.01"/>
+            </geometry>
+            <material name="blue"/>
+        </collision>
+        <!-- <xacro:inertial_cylinder mass="0.1" radius="0.05" length="0.04">
+            <origin xyz="0 0 0" rpy="0 0 0"/>
+        </xacro:inertial_cylinder> -->
+    </link>
+    <!-- ANKLE_PITCH LINK -->
+    <joint name="ankle_pitch_joint" type="continuous">
+        <parent link="ankle_yaw"/>
+        <child link="ankle_pitch"/>
+        <origin xyz="0 0 0" rpy="${pi/2} 0 0"/>
+        <axis xyz="0 0 1"/>
+    </joint>
+    <link name="ankle_pitch">
+        <visual>
+            <geometry>
+                <cylinder radius="0.01" length="0.01"/>
             </geometry>
             <material name="black"/>
@@ -105,11 +83,185 @@
         <collision>
             <geometry>
-                <sphere radius="0.05"/>
+                <cylinder radius="0.01" length="0.01"/>
             </geometry>
             <material name="black"/>
         </collision>
-        <xacro:inertial_sphere mass="0.1" radius="0.05">
-            <origin xyz="0 0 0" rpy="0 0 0"/>
-        </xacro:inertial_sphere>
+        <!-- <xacro:inertial_cylinder mass="0.1" radius="0.05" length="0.04">
+            <origin xyz="0 0 0" rpy="0 0 0"/>
+        </xacro:inertial_cylinder> -->
+    </link>
+    <!-- CALF LINK -->
+    <joint name="calf_joint" type="fixed">
+        <parent link="ankle_pitch"/>
+        <child link="calf"/>
+        <origin xyz="0 0 0" rpy="-${pi/2} 0 0"/>
+        <axis xyz="0 0 1"/>
+    </joint>
+    <link name="calf">
+        <visual>
+            <origin xyz="0 0 0.2" rpy="0 0 0"/>
+            <geometry>
+                <cylinder radius="0.025" length="0.4"/>
+            </geometry>
+            <material name="white"/>
+        </visual>
+        <collision>
+            <origin xyz="0 0 0.2" rpy="0 0 0"/>
+            <geometry>
+                <cylinder radius="0.025" length="0.4"/>
+            </geometry>
+            <material name="white"/>
+        </collision>
+        <!-- <xacro:inertial_cylinder mass="0.1" radius="0.05" length="0.04">
+            <origin xyz="0 0 0" rpy="0 0 0"/>
+        </xacro:inertial_cylinder> -->
+    </link>
+    <!-- KNEE LINK -->
+    <joint name="knee_joint" type="continuous">
+        <parent link="calf"/>
+        <child link="knee"/>
+        <origin xyz="0 0 0.4" rpy="${pi/2} 0 0"/>
+        <axis xyz="0 0 1"/>
+    </joint>
+    <link name="knee">
+        <visual>
+            <geometry>
+                <cylinder radius="0.01" length="0.01"/>
+            </geometry>
+            <material name="blue"/>
+        </visual>
+        <collision>
+            <geometry>
+                <cylinder radius="0.01" length="0.01"/>
+            </geometry>
+            <material name="blue"/>
+        </collision>
+        <!-- <xacro:inertial_cylinder mass="0.1" radius="0.05" length="0.04">
+            <origin xyz="0 0 0" rpy="0 0 0"/>
+        </xacro:inertial_cylinder> -->
+    </link>
+    <!-- THIGH LINK -->
+    <joint name="thigh_joint" type="fixed">
+        <parent link="knee"/>
+        <child link="tight"/>
+        <origin xyz="0 0 0" rpy="-${pi/2} 0 0"/>
+        <axis xyz="0 0 1"/>
+    </joint>
+    <link name="tight">
+        <visual>
+            <origin xyz="0 0 0.2" rpy="0 0 0"/>
+            <geometry>
+                <cylinder radius="0.025" length="0.4"/>
+            </geometry>
+            <material name="white"/>
+        </visual>
+        <collision>
+            <origin xyz="0 0 0.2" rpy="0 0 0"/>
+            <geometry>
+                <cylinder radius="0.025" length="0.4"/>
+            </geometry>
+            <material name="white"/>
+        </collision>
+        <!-- <xacro:inertial_cylinder mass="0.1" radius="0.05" length="0.04">
+            <origin xyz="0 0 0" rpy="0 0 0"/>
+        </xacro:inertial_cylinder> -->
+    </link>
+    <!-- HIP_YAW LINK -->
+    <joint name="hip_yaw_joint" type="continuous">
+        <parent link="tight"/>
+        <child link="hip_yaw"/>
+        <origin xyz="0 0 0.4" rpy="0 0 0"/>
+        <axis xyz="0 0 1"/>
+    </joint>
+    <link name="hip_yaw">
+        <visual>
+            <geometry>
+                <cylinder radius="0.01" length="0.01"/>
+            </geometry>
+            <material name="blue"/>
+        </visual>
+        <collision>
+            <geometry>
+                <cylinder radius="0.01" length="0.01"/>
+            </geometry>
+            <material name="blue"/>
+        </collision>
+        <!-- <xacro:inertial_cylinder mass="0.1" radius="0.05" length="0.04">
+            <origin xyz="0 0 0" rpy="0 0 0"/>
+        </xacro:inertial_cylinder> -->
+    </link>
+    <!-- HIP_PITCH LINK -->
+    <joint name="hip_pitch_joint" type="continuous">
+        <parent link="hip_yaw"/>
+        <child link="hip_pitch"/>
+        <origin xyz="0 0 0" rpy="${pi/2} 0 0"/>
+        <axis xyz="0 0 1"/>
+    </joint>
+    <link name="hip_pitch">
+        <visual>
+            <geometry>
+                <cylinder radius="0.01" length="0.01"/>
+            </geometry>
+            <material name="blue"/>
+        </visual>
+        <collision>
+            <geometry>
+                <cylinder radius="0.01" length="0.01"/>
+            </geometry>
+            <material name="blue"/>
+        </collision>
+        <!-- <xacro:inertial_cylinder mass="0.1" radius="0.05" length="0.04">
+            <origin xyz="0 0 0" rpy="0 0 0"/>
+        </xacro:inertial_cylinder> -->
+    </link>
+    <!-- HIP_ROLL LINK -->
+    <joint name="hip_roll_joint" type="continuous">
+        <parent link="hip_pitch"/>
+        <child link="hip_roll"/>
+        <origin xyz="0 0 0" rpy="-${pi/2} 0 0"/>
+        <axis xyz="1 0 0"/>
+    </joint>
+    <link name="hip_roll">
+        <visual>
+            <geometry>
+                <cylinder radius="0.01" length="0.01"/>
+            </geometry>
+            <material name="blue"/>
+        </visual>
+        <collision>
+            <geometry>
+                <cylinder radius="0.01" length="0.01"/>
+            </geometry>
+            <material name="blue"/>
+        </collision>
+        <!-- <xacro:inertial_cylinder mass="0.1" radius="0.05" length="0.04">
+            <origin xyz="0 0 0" rpy="0 0 0"/>
+        </xacro:inertial_cylinder> -->
+    </link>
+    <!-- WAIST LINK -->
+    <joint name="waist_joint" type="fixed">
+        <parent link="hip_roll"/>
+        <child link="waist"/>
+        <origin xyz="0 0 0" rpy="0 0 0"/>
+        <axis xyz="0 0 1"/>
+    </joint>
+    <link name="waist">
+        <visual>
+            <origin xyz="0 0 0.157"/>
+            <geometry>
+                <box size="0.1 0.1 0.314"/>
+            </geometry>
+            <material name="white"/>
+        </visual>
+        <collision>
+            <origin xyz="0 0 0.157"/>
+            <geometry>
+                <box size="0.1 0.1 0.314"/>
+            </geometry>
+            <material name="white"/>
+        </collision>
+        <!-- <xacro:inertial_box mass="0.5" x="0.3" y="0.3" z="0.15"> -->
+            <!-- <origin xyz="0.15 0 0.075" rpy="0 0 0"/> -->
+        <!-- </xacro:inertial_box> -->
     </link>
 </robot>

Commit message: ankle roll modify

File: description/robot_core.xacro (robot description, xacro)
@@ -43,12 +43,12 @@
         <!-- </xacro:inertial_box> -->
     </link>
-    <!-- ANKLE_YAW LINK -->
-    <joint name="ankle_yaw_joint" type="continuous">
+    <!-- ANKLE_ROLL LINK -->
+    <joint name="ankle_roll_joint" type="continuous">
         <parent link="foot"/>
-        <child link="ankle_yaw"/>
-        <origin xyz="-0.01 0 0.01" rpy="0 0 0"/>
-        <axis xyz="0 0 1"/>
-    </joint>
-    <link name="ankle_yaw">
+        <child link="ankle_roll"/>
+        <origin xyz="-0.01 0 0.01" rpy="0 ${pi/2} 0"/>
+        <axis xyz="0 0 1"/>
+    </joint>
+    <link name="ankle_roll">
         <visual>
             <geometry>
@@ -69,7 +69,7 @@
     <!-- ANKLE_PITCH LINK -->
     <joint name="ankle_pitch_joint" type="continuous">
-        <parent link="ankle_yaw"/>
+        <parent link="ankle_roll"/>
         <child link="ankle_pitch"/>
-        <origin xyz="0 0 0" rpy="${pi/2} 0 0"/>
+        <origin xyz="0 0 0" rpy="${pi/2} -${pi/2} 0"/>
         <axis xyz="0 0 1"/>
     </joint>
